Commit message: Fixing bugs with the Barrel Detector.
Edited mistii.urdf and changed the camera roll. NOTE THAT NO NODES THAT USE A CAMERA TRANSFORM WILL WORK ANYMORE.

File: igvc/launch/mistii.urdf (robot description, URDF)
Before this commit: robot test_platform, 8 links, 7 joints
Joints:
- joint camera: origin xyz=0 -0.18 1.34 rpy=-0.3491 0 0 -> xyz=0 -0.18 1.34 rpy=-1.9198 0 0
